File: hardware/circuit/circuit-board.brd (EAGLE design)
At the start: 20.3 x 73.7 mm, 14 parts, among them U1 ADUM1200CRZ

Commit message: Added missing 100k resistor to base of PN2222A, deleted flawed Gerber files - board layout is not updated for now because I have V2 in mind and PCBs in hand already
Parts:
- added R4: 100k, SparkFun-Resistors:0603
Connections:
- new net N$2: NP2222A.B, R4.2
- net PWR-CTRL: now also R4.1; no longer NP2222A.B
Routing:
- net PWR-CTRL: track 25.4 -> 22.8 mm
Changed lines of the file:
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@@
 <element name="EXT-GND" library="wirepad" package="5-2,5" value="WIREPADSMD5-2,5" x="7.62" y="10.16"/>
 <element name="LED-GND" library="wirepad" package="5-2,5" value="WIREPADSMD5-2,5" x="3.81" y="17.78" rot="R270"/>
+<element name="R4" library="SparkFun-Resistors" package="0603" value="100k" x="-3.81" y="0">
+<attribute name="PROD_ID" value="RES-07828" x="-3.81" y="0" size="1.778" layer="27" display="off"/>
+</element>
 </elements>
 <signals>
@@
 <contactref element="OK1" pad="5"/>
 <contactref element="IRLB8721" pad="G"/>
-<contactref element="NP2222A" pad="B"/>
 <wire x1="10.9728" y1="22.4028" x2="8.89" y2="20.32" width="0.254" layer="1"/>
 <wire x1="5.2578" y1="33.8328" x2="5.2578" y2="34.29" width="0.254" layer="16"/>
@@
 <wire x1="12.3444" y1="32.2326" x2="11.8872" y2="31.7754" width="0.254" layer="16"/>
 <wire x1="13.4874" y1="32.2326" x2="12.3444" y2="32.2326" width="0.254" layer="16"/>
-<wire x1="15.24" y1="30.48" x2="13.4874" y2="32.2326" width="0.254" layer="16"/>
 <wire x1="5.2578" y1="34.29" x2="5.08" y2="34.29" width="0.254" layer="16"/>
 <wire x1="11.2014" y1="25.3746" x2="15.0876" y2="29.2608" width="0.254" layer="1"/>
-<wire x1="15.24" y1="30.48" x2="15.0876" y2="30.48" width="0.254" layer="1"/>
 <wire x1="15.0876" y1="30.48" x2="15.0876" y2="29.2608" width="0.254" layer="1"/>
 <wire x1="11.2014" y1="24.13" x2="11.01" y2="24.13" width="0.254" layer="1"/>
@@
 <wire x1="11.01" y1="24.13" x2="10.9728" y2="24.13" width="0.254" layer="1"/>
 <wire x1="10.9728" y1="24.13" x2="10.9728" y2="22.4028" width="0.254" layer="1"/>
+<contactref element="R4" pad="1"/>
+<wire x1="15.0876" y1="30.48" x2="13.4874" y2="32.2326" width="0" layer="19" extent="1-16"/>
+<wire x1="-4.66" y1="0" x2="8.89" y2="20.32" width="0" layer="19" extent="1-1"/>
 </signal>
 <signal name="N$3">
@@
 <wire x1="14.4018" y1="35.6362" x2="14.4018" y2="36.3474" width="0.254" layer="1"/>
 </signal>
+<signal name="N$2">
+<contactref element="NP2222A" pad="B"/>
+<contactref element="R4" pad="2"/>
+<wire x1="-2.96" y1="0" x2="15.24" y2="30.48" width="0" layer="19" extent="1-1"/>
+</signal>
 </signals>
